File: aquariumUnit_v2/aquariumUnit_v2.kicad_pcb (KiCad board)
At the start: 2 copper layers, 9 parts, among them P1 ESP_PROG, U1 ESP-12E

Commit message: update aquarium
Parts:
- added D1: D, Diodes_ThroughHole:Diode_DO-35_SOD27_Horizontal_RM10, F.Cu at (48.3, 71.1)
- added D2: D, Diodes_ThroughHole:Diode_DO-35_SOD27_Horizontal_RM10, F.Cu at (27.9, 71.1)
- added P2: PUMP, Pin_Headers:Pin_Header_Straight_1x02, F.Cu at (53.3, 74.9)
- added P3: POWER, Connect:AK300-2, F.Cu at (27.9, 27.9)
- added P4: BUTTONS, Pin_Headers:Pin_Header_Straight_1x03, F.Cu at (76.2, 50.8)
- added P5: FAN, Pin_Headers:Pin_Header_Straight_1x02, F.Cu at (33.0, 74.9)
- added P6: DS, Pin_Headers:Pin_Header_Straight_1x03, F.Cu at (76.2, 38.1)
- added P7: SUB_LEDS, Pin_Headers:Pin_Header_Straight_1x04, F.Cu at (22.9, 64.8)
- added P8: LED_STRIP, Connect:AK300-2, F.Cu at (76.2, 78.7)
- added Q1: PUMP_MOS, TO_SOT_Packages_THT:TO-220_Neutral123_Vertical, F.Cu at (43.2, 76.2)
- added Q2: FAN_MOS, TO_SOT_Packages_THT:TO-220_Neutral123_Vertical, F.Cu at (22.9, 76.2)
- added Q3: LED_MOS, TO_SOT_Packages_THT:TO-220_Neutral123_Vertical, F.Cu at (63.5, 76.2)
- added R7: 330, Resistors_ThroughHole:Resistor_Vertical_RM5mm, F.Cu at (50.8, 30.5)
- added R8: 560, Resistors_ThroughHole:Resistor_Vertical_RM5mm, F.Cu at (63.5, 30.5)
- added R9: 470, Resistors_SMD:R_1210_HandSoldering, F.Cu at (33.0, 64.8)
- added U2: LM317T, Power_Integrations:TO-220, F.Cu at (40.6, 30.5)
- added U3: ULN2003, SMD_Packages:SO-16-N, F.Cu at (33.0, 57.1)
- P1: value ESP_PROG -> SERVO; footprint Pin_Headers:Pin_Header_Straight_1x05 -> Pin_Headers:Pin_Header_Straight_1x03
- R5: value 470 -> 10K
- R6: value 470 -> 4.7K
- moved P1 50.9 mm to (22.9, 45.7)
- moved R3 12.7 mm to (33.0, 44.5), turned to 270 degrees
Connections:
- P1 pad 1: /RX -> /D16
- P1 pad 2: /TX -> +3V3
- R1 pad 2: /DTR -> /D0
- R5 pad 1: /DTR -> /D2
- R5 pad 2: /D0 -> GND
- R6 pad 1: /RST -> +3V3
- R6 pad 2: /D16 -> /D0
Routing:
- net +3V3: track 33.9 -> 177.0 mm
- net GND: track 63.7 -> 202.4 mm
- net +12V: track 0.00 -> 112.5 mm
- net /D0: track 16.9 -> 120.6 mm, vias 0 -> 2
- net /D5: track 0.00 -> 81.4 mm, vias 0 -> 1
- net /D4: track 0.00 -> 69.9 mm, vias 0 -> 1
- net /RST: track 50.6 -> 14.0 mm
- net /DTR: track 32.5 -> 0.00 mm
- net /D2: track 0.00 -> 27.6 mm, vias 0 -> 1
- net /D9: track 0.00 -> 26.1 mm, vias 0 -> 1
- net /D15: track 14.5 -> 36.3 mm
- net Net-(R7-Pad2): track 0.00 -> 21.4 mm
- net /D16: track 7.13 -> 28.3 mm
- net Net-(P8-Pad2): track 0.00 -> 14.9 mm
- net /D13: track 0.00 -> 14.8 mm
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Other:
- net class Default: clearance 0.4 -> 0.6; trace_width 0.6 -> 0.8; via_dia 1.2 -> 2
- rule trace_clearance: 0.4 -> 0.6
- board text added: "Aquarium unit v2"
