File: aquariumUnit_v2/aquariumUnit_v2.sch (KiCad schematic (older format))
At the start: 22 parts, among them U1 ESP-12E

Commit message: update aquarium
Parts:
- removed Q?: BC557, TO-92, symbol BC557
- added P8: LED_STRIP, Connect:AK300-2, symbol CONN_01X02
- added Q3: LED_MOS, TO_SOT_Packages_THT:TO-220_Neutral123_Vertical, symbol Q_NMOS_DSG
- added R6: 4.7K, Resistors_SMD:R_1210_HandSoldering, symbol R
- added R9: 470, Resistors_SMD:R_1210_HandSoldering, symbol R
- added U3: ULN2003, SMD_Packages:SO-16-N, symbol ULN2003
- D1, D2: renamed from D?; footprint (none) -> Diodes_ThroughHole:Diode_DO-35_SOD27_Horizontal_RM10
- P1, P6: renamed from P?; footprint (none) -> Pin_Headers:Pin_Header_Straight_1x03
- P2, P5: renamed from P?; footprint (none) -> Pin_Headers:Pin_Header_Straight_1x02
- P3: renamed from P?; footprint (none) -> Connect:AK300-2
- P4: renamed from P?; value CONN_01X03 -> BUTTONS; footprint (none) -> Pin_Headers:Pin_Header_Straight_1x03
- P7: renamed from P?; value CONN_01X04 -> SUB_LEDS; footprint (none) -> Pin_Headers:Pin_Header_Straight_1x04
- Q1, Q2: renamed from Q?; footprint (none) -> TO_SOT_Packages_THT:TO-220_Neutral123_Vertical
- R7, R8: renamed from R?; footprint (none) -> Resistors_ThroughHole:Resistor_Vertical_RM5mm
- U2: renamed from U?; footprint TO-220 -> Power_Integrations:TO-220
- gave numbers to parts that had none: 1
Connections:
- net labels removed: B_GND, DS, FEED, G_GND, R_GND
- wire segments 28 -> 40
- no-connect marks 4 -> 13
Other:
- moved on the sheet: P7
