File: aquariumUnit_v2/aquariumUnit_v2.1.kicad_pcb (KiCad board)
At the start: 2 copper layers, 23 parts, among them P1 SERVO, P2 PUMP, P3 POWER, P4 BUTTONS, P5 FAN, P6 DS, P7 SUB_LEDS, P8 LED_STRIP, U1 ESP-12E, U2 LM317T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

Commit message: hude update
Routing:
- net +3V3: track 160.4 -> 0.00 mm
- net GND: track 151.5 -> 0.00 mm
- net +12V: track 109.4 -> 44.1 mm
- net /D0: track 43.9 -> 0.00 mm
- net /D2: track 35.2 -> 0.00 mm
- net /BT1: track 34.3 -> 0.00 mm
- net Net-(P8-Pad2): track 23.1 -> 0.00 mm
- net /BT2: track 22.2 -> 0.00 mm
- net Net-(R7-Pad2): track 21.9 -> 0.00 mm
- net Net-(P7-Pad4): track 18.1 -> 0.00 mm
- net Net-(P7-Pad3): track 15.6 -> 0.00 mm
- net Net-(P7-Pad2): track 14.3 -> 0.00 mm
- net /D15: track 14.0 -> 0.00 mm
- net Net-(P5-Pad2): track 11.4 -> 0.00 mm
- net Net-(P2-Pad2): track 11.4 -> 0.00 mm
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