File: aquariumUnit_v2/aquariumUnit_v2.1.sch (KiCad schematic (older format))
At the start: 23 parts, among them P1 SERVO, P2 PUMP, P3 POWER, P4 BUTTONS, P5 FAN, P6 DS, P7 SUB_LEDS, P8 LED_STRIP, U1 ESP-12E, U2 LM317T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

Commit message: hude update
Parts:
- U1: symbol ESP-12E -> ESP-12E-RESCUE-aquariumUnit_v2.1
Connections:
- net labels removed: D10, D9
- no-connect marks 4 -> 6
Changed lines of the file:
@@
 EESchema Schematic File Version 2
+LIBS:aquariumUnit_v2.1-rescue
 LIBS:power
 LIBS:device
@@
 $EndDescr
 $Comp
-L ESP-12E U1
+L ESP-12E-RESCUE-aquariumUnit_v2.1 U1
 U 1 1 574FE884
 P 2600 1600
@@
 Text Label 3500 1400 0    60   ~ 0
 TX
-Text Label 2550 2500 3    60   ~ 0
-D9
-Text Label 2650 2500 3    60   ~ 0
-D10
 Text Label 1700 1600 0    60   ~ 0
 D16
@@
 D13
 Text Label 1500 4850 0    60   ~ 0
-D9
+RX
 Text Label 1500 4950 0    60   ~ 0
-D10
+TX
 Text Label 1500 5050 0    60   ~ 0
 D15
@@
 Wire Wire Line
 	1500 5150 1950 5150
+NoConn ~ 2550 2500
+NoConn ~ 2650 2500
 $EndSCHEMATC
